Commit message: robot model description slam

File: src/tadeocar_description/urdf/tadeocar_control.urdf.xacro (robot description, xacro)
@@ -11,66 +11,99 @@
   <link name="base_link">
     <inertial>
-      <mass value="20.0"/>
-      <origin xyz="0 0 0" rpy="0 0 0"/>
-      <inertia ixx="1.0" ixy="0.0" ixz="0.0" iyy="1.0" iyz="0.0" izz="1.0"/>
+      <mass value="50.0"/>
+      <origin xyz="0 0 0" rpy="0 0 0"/>
+      <inertia ixx="4.0" ixy="0.0" ixz="0.0" iyy="4.0" iyz="0.0" izz="2.0"/>
     </inertial>
+    <visual>
+      <origin xyz="0 0 0.155" rpy="0 0 0"/>
+      <geometry>
+        <mesh filename="package://tadeocar_description/models/tadeocar_v1/meshes/chassis/chasis_base.dae" scale="1 1 1"/>
+      </geometry>
+    </visual>
   </link>
   <!-- Chassis Link -->
   <link name="chasis_link">
     <inertial>
-      <mass value="15.0"/>
-      <origin xyz="0 0 0" rpy="0 0 0"/>
-      <inertia ixx="0.5" ixy="0.0" ixz="0.0" iyy="0.5" iyz="0.0" izz="0.5"/>
+      <mass value="20.0"/>
+      <origin xyz="0 0 0" rpy="0 0 0"/>
+      <inertia ixx="1.0" ixy="0.0" ixz="0.0" iyy="1.0" iyz="0.0" izz="0.5"/>
     </inertial>
+    <visual>
+      <origin xyz="-0.49 0.39 -0.126" rpy="1.5708 0 3.14159"/>
+      <geometry>
+        <mesh filename="package://tadeocar_description/models/tadeocar_v1/meshes/chassis/chasis.dae" scale="0.001 0.001 0.001"/>
+      </geometry>
+    </visual>
   </link>
   <joint name="chasis_joint" type="fixed">
     <parent link="base_link"/>
     <child link="chasis_link"/>
-    <origin xyz="0 0 0" rpy="0 0 0"/>
+    <origin xyz="0 0 0.35" rpy="0 0 0"/>
   </joint>
   <!-- LiDAR Link -->
-  <link name="base_scan"/>
+  <link name="base_scan">
+    <inertial>
+      <mass value="0.125"/>
+      <origin xyz="0 0 0" rpy="0 0 0"/>
+      <inertia ixx="0.001" ixy="0.0" ixz="0.0" iyy="0.001" iyz="0.0" izz="0.001"/>
+    </inertial>
+    <visual>
+      <origin xyz="0 0 0" rpy="0 0 0"/>
+      <geometry>
+        <cylinder radius="0.035" length="0.030"/>
+      </geometry>
+      <material name="lidar_color">
+        <color rgba="0.1 0.1 0.1 1.0"/>
+      </material>
+    </visual>
+  </link>
   <joint name="lidar_joint" type="fixed">
     <parent link="base_link"/>
     <child link="base_scan"/>
-    <origin xyz="0 0 0.30" rpy="0 0 0"/>
+    <origin xyz="0.55 0 0.33" rpy="0 0 0"/>
   </joint>
   <!-- Steering Links -->
-  <xacro:macro name="steering_link" params="prefix">
+  <xacro:macro name="steering_link" params="prefix reflect_yaw">
     <link name="${prefix}_steering_link">
       <inertial>
-        <mass value="0.5"/>
+        <mass value="2.0"/>
         <origin xyz="0 0 0" rpy="0 0 0"/>
         <inertia ixx="0.01" ixy="0.0" ixz="0.0" iyy="0.01" iyz="0.0" izz="0.01"/>
       </inertial>
+      <visual>
+        <origin xyz="0 0 0.227" rpy="0 3.14159 ${reflect_yaw}"/>
+        <geometry>
+          <mesh filename="package://tadeocar_description/models/tadeocar_v1/meshes/suspension/suspension.dae" scale="1 1 1"/>
+        </geometry>
+      </visual>
     </link>
   </xacro:macro>
-  <xacro:steering_link prefix="front_left"/>
-  <xacro:steering_link prefix="front_right"/>
-  <xacro:steering_link prefix="rear_left"/>
-  <xacro:steering_link prefix="rear_right"/>
+  <xacro:steering_link prefix="front_left" reflect_yaw="3.14159"/>
+  <xacro:steering_link prefix="front_right" reflect_yaw="-3.14159"/>
+  <xacro:steering_link prefix="rear_left" reflect_yaw="0"/>
+  <xacro:steering_link prefix="rear_right" reflect_yaw="0"/>
   <!-- Steering Joints -->
   <joint name="front_left_steering_joint" type="continuous">
-    <parent link="chasis_link"/>
+    <parent link="base_link"/>
     <child link="front_left_steering_link"/>
-    <origin xyz="0.3 0.25 0" rpy="0 0 0"/>
+    <origin xyz="0.478 0.275 0" rpy="0 0 0"/>
     <axis xyz="0 0 1"/>
   </joint>
   <joint name="front_right_steering_joint" type="continuous">
-    <parent link="chasis_link"/>
+    <parent link="base_link"/>
     <child link="front_right_steering_link"/>
-    <origin xyz="0.3 -0.25 0" rpy="0 0 0"/>
+    <origin xyz="0.478 -0.275 0" rpy="0 0 0"/>
     <axis xyz="0 0 1"/>
   </joint>
   <joint name="rear_left_steering_joint" type="continuous">
-    <parent link="chasis_link"/>
+    <parent link="base_link"/>
     <child link="rear_left_steering_link"/>
-    <origin xyz="-0.3 0.25 0" rpy="0 0 0"/>
+    <origin xyz="-0.58 0.275 0" rpy="0 0 0"/>
     <axis xyz="0 0 1"/>
   </joint>
   <joint name="rear_right_steering_joint" type="continuous">
-    <parent link="chasis_link"/>
+    <parent link="base_link"/>
     <child link="rear_right_steering_link"/>
-    <origin xyz="-0.3 -0.25 0" rpy="0 0 0"/>
+    <origin xyz="-0.58 -0.275 0" rpy="0 0 0"/>
     <axis xyz="0 0 1"/>
   </joint>
@@ -79,8 +112,14 @@
     <link name="${prefix}_wheel_link">
       <inertial>
-        <mass value="1.0"/>
+        <mass value="3.0"/>
         <origin xyz="0 0 0" rpy="0 0 0"/>
-        <inertia ixx="0.02" ixy="0.0" ixz="0.0" iyy="0.02" iyz="0.0" izz="0.02"/>
+        <inertia ixx="0.1" ixy="0.0" ixz="0.0" iyy="0.1" iyz="0.0" izz="0.1"/>
       </inertial>
+      <visual>
+        <origin xyz="0 0 0" rpy="1.5708 0 0"/>
+        <geometry>
+          <mesh filename="package://tadeocar_description/models/tadeocar_v1/meshes/wheels/wheel.dae" scale="1 1 1"/>
+        </geometry>
+      </visual>
     </link>
   </xacro:macro>
@@ -93,5 +132,5 @@
     <parent link="front_left_steering_link"/>
     <child link="front_left_wheel_link"/>
-    <origin xyz="0 0 -0.1" rpy="0 0 0"/>
+    <origin xyz="0.05 0 0" rpy="0 0 0"/>
     <axis xyz="0 1 0"/>
   </joint>
@@ -99,5 +138,5 @@
     <parent link="front_right_steering_link"/>
     <child link="front_right_wheel_link"/>
-    <origin xyz="0 0 -0.1" rpy="0 0 0"/>
+    <origin xyz="0.05 0 0" rpy="0 0 0"/>
     <axis xyz="0 1 0"/>
   </joint>
@@ -105,5 +144,5 @@
     <parent link="rear_left_steering_link"/>
     <child link="rear_left_wheel_link"/>
-    <origin xyz="0 0 -0.1" rpy="0 0 0"/>
+    <origin xyz="-0.05 0 0" rpy="0 0 0"/>
     <axis xyz="0 1 0"/>
   </joint>
@@ -111,5 +150,5 @@
     <parent link="rear_right_steering_link"/>
     <child link="rear_right_wheel_link"/>
-    <origin xyz="0 0 -0.1" rpy="0 0 0"/>
+    <origin xyz="-0.05 0 0" rpy="0 0 0"/>
     <axis xyz="0 1 0"/>
   </joint>

Commit message: camera estereo

File: src/tadeocar_description/urdf/tadeocar_control.urdf.xacro (robot description, xacro)
@@ -62,4 +62,101 @@
     <child link="base_scan"/>
     <origin xyz="0.55 0 0.33" rpy="0 0 0"/>
+  </joint>
+  <!-- Stereo Camera Base Link -->
+  <link name="stereo_camera_base">
+    <inertial>
+      <mass value="0.1"/>
+      <origin xyz="0 0 0" rpy="0 0 0"/>
+      <inertia ixx="0.0001" ixy="0.0" ixz="0.0" iyy="0.0001" iyz="0.0" izz="0.0001"/>
+    </inertial>
+    <visual>
+      <origin xyz="0 0 0" rpy="0 0 1.5708"/>
+      <geometry>
+        <box size="0.15 0.05 0.03"/>
+      </geometry>
+      <material name="camera_color">
+        <color rgba="0.2 0.2 0.2 1.0"/>
+      </material>
+    </visual>
+    <collision>
+      <origin xyz="0 0 0" rpy="0 0 1.5708"/>
+      <geometry>
+        <box size="0.15 0.05 0.03"/>
+      </geometry>
+    </collision>
+  </link>
+  <joint name="stereo_camera_base_joint" type="fixed">
+    <parent link="base_link"/>
+    <child link="stereo_camera_base"/>
+    <origin xyz="0.55 0 0.40" rpy="0 0 0"/>
+  </joint>
+  <!-- Left Camera Link -->
+  <link name="camera_left">
+    <inertial>
+      <mass value="0.05"/>
+      <origin xyz="0 0 0" rpy="0 0 0"/>
+      <inertia ixx="0.00001" ixy="0.0" ixz="0.0" iyy="0.00001" iyz="0.0" izz="0.00001"/>
+    </inertial>
+    <visual>
+      <origin xyz="0 0 0" rpy="0 1.5708 0"/>
+      <geometry>
+        <cylinder radius="0.01" length="0.01"/>
+      </geometry>
+      <material name="camera_lens">
+        <color rgba="0.1 0.1 0.1 1.0"/>
+      </material>
+    </visual>
+    <collision>
+      <origin xyz="0 0 0" rpy="0 1.5708 0"/>
+      <geometry>
+        <cylinder radius="0.01" length="0.01"/>
+      </geometry>
+    </collision>
+  </link>
+  <joint name="camera_left_joint" type="fixed">
+    <parent link="stereo_camera_base"/>
+    <child link="camera_left"/>
+    <origin xyz="0.03 0.06 0" rpy="0 0 0"/>
+  </joint>
+  <!-- Right Camera Link -->
+  <link name="camera_right">
+    <inertial>
+      <mass value="0.05"/>
+      <origin xyz="0 0 0" rpy="0 0 0"/>
+      <inertia ixx="0.00001" ixy="0.0" ixz="0.0" iyy="0.00001" iyz="0.0" izz="0.00001"/>
+    </inertial>
+    <visual>
+      <origin xyz="0 0 0" rpy="0 1.5708 0"/>
+      <geometry>
+        <cylinder radius="0.01" length="0.01"/>
+      </geometry>
+      <material name="camera_lens">
+        <color rgba="0.1 0.1 0.1 1.0"/>
+      </material>
+    </visual>
+    <collision>
+      <origin xyz="0 0 0" rpy="0 1.5708 0"/>
+      <geometry>
+        <cylinder radius="0.01" length="0.01"/>
+      </geometry>
+    </collision>
+  </link>
+  <joint name="camera_right_joint" type="fixed">
+    <parent link="stereo_camera_base"/>
+    <child link="camera_right"/>
+    <origin xyz="0.03 -0.06 0" rpy="0 0 0"/>
+  </joint>
+  <!-- Camera Optical Frames (for image topics) -->
+  <link name="camera_left_optical"/>
+  <joint name="camera_left_optical_joint" type="fixed">
+    <parent link="camera_left"/>
+    <child link="camera_left_optical"/>
+    <origin xyz="0.005 0 0" rpy="-1.5708 0 -1.5708"/>
+  </joint>
+  <link name="camera_right_optical"/>
+  <joint name="camera_right_optical_joint" type="fixed">
+    <parent link="camera_right"/>
+    <child link="camera_right_optical"/>
+    <origin xyz="0.005 0 0" rpy="-1.5708 0 -1.5708"/>
   </joint>
   <!-- Steering Links -->
@@ -237,3 +334,84 @@
     </plugin>
   </gazebo>
+  <!-- Gazebo properties for stereo camera base -->
+  <gazebo reference="stereo_camera_base">
+    <gravity>false</gravity>
+    <kinematic>true</kinematic>
+  </gazebo>
+  <!-- Gazebo properties for left camera -->
+  <gazebo reference="camera_left">
+    <gravity>false</gravity>
+    <kinematic>true</kinematic>
+  </gazebo>
+  <!-- Gazebo properties for right camera -->
+  <gazebo reference="camera_right">
+    <gravity>false</gravity>
+    <kinematic>true</kinematic>
+  </gazebo>
+  <!-- Gazebo plugin for left camera -->
+  <gazebo reference="camera_left">
+    <sensor type="camera" name="camera_left_sensor">
+      <update_rate>30.0</update_rate>
+      <camera name="left">
+        <horizontal_fov>1.3962634</horizontal_fov>
+        <image>
+          <width>1280</width>
+          <height>720</height>
+          <format>R8G8B8</format>
+        </image>
+        <clip>
+          <near>0.02</near>
+          <far>300</far>
+        </clip>
+        <noise>
+          <type>gaussian</type>
+          <mean>0.0</mean>
+          <stddev>0.007</stddev>
+        </noise>
+      </camera>
+      <plugin name="camera_left_controller" filename="libgazebo_ros_camera.so">
+        <ros>
+          <namespace>/</namespace>
+          <remapping>~/image_raw:=camera/left/image_raw</remapping>
+          <remapping>~/camera_info:=camera/left/camera_info</remapping>
+        </ros>
+        <camera_name>camera_left</camera_name>
+        <frame_name>camera_left_optical</frame_name>
+        <hack_baseline>0.12</hack_baseline>
+      </plugin>
+    </sensor>
+  </gazebo>
+  <!-- Gazebo plugin for right camera -->
+  <gazebo reference="camera_right">
+    <sensor type="camera" name="camera_right_sensor">
+      <update_rate>30.0</update_rate>
+      <camera name="right">
+        <horizontal_fov>1.3962634</horizontal_fov>
+        <image>
+          <width>1280</width>
+          <height>720</height>
+          <format>R8G8B8</format>
+        </image>
+        <clip>
+          <near>0.02</near>
+          <far>300</far>
+        </clip>
+        <noise>
+          <type>gaussian</type>
+          <mean>0.0</mean>
+          <stddev>0.007</stddev>
+        </noise>
+      </camera>
+      <plugin name="camera_right_controller" filename="libgazebo_ros_camera.so">
+        <ros>
+          <namespace>/</namespace>
+          <remapping>~/image_raw:=camera/right/image_raw</remapping>
+          <remapping>~/camera_info:=camera/right/camera_info</remapping>
+        </ros>
+        <camera_name>camera_right</camera_name>
+        <frame_name>camera_right_optical</frame_name>
+        <hack_baseline>0.12</hack_baseline>
+      </plugin>
+    </sensor>
+  </gazebo>
 </robot>

Commit message: navigation2

File: src/tadeocar_description/urdf/tadeocar_control.urdf.xacro (robot description, xacro)
@@ -149,7 +149,7 @@
     <link name="${prefix}_steering_link">
       <inertial>
-        <mass value="2.0"/>
+        <mass value="6.0"/>
         <origin xyz="0 0 0" rpy="0 0 0"/>
-        <inertia ixx="0.01" ixy="0.0" ixz="0.0" iyy="0.01" iyz="0.0" izz="0.01"/>
+        <inertia ixx="0.05" ixy="0.0" ixz="0.0" iyy="0.05" iyz="0.0" izz="0.05"/>
       </inertial>
       <visual>
@@ -159,4 +159,10 @@
         </geometry>
       </visual>
+      <collision>
+        <origin xyz="0 0 0.227" rpy="0 3.14159 ${reflect_yaw}"/>
+        <geometry>
+          <mesh filename="package://tadeocar_description/models/tadeocar_v1/meshes/suspension/suspension.dae" scale="1 1 1"/>
+        </geometry>
+      </collision>
     </link>
   </xacro:macro>
@@ -171,4 +177,5 @@
     <origin xyz="0.478 0.275 0" rpy="0 0 0"/>
     <axis xyz="0 0 1"/>
+    <dynamics damping="5.0" friction="0.1"/>
   </joint>
   <joint name="front_right_steering_joint" type="continuous">
@@ -177,4 +184,5 @@
     <origin xyz="0.478 -0.275 0" rpy="0 0 0"/>
     <axis xyz="0 0 1"/>
+    <dynamics damping="5.0" friction="0.1"/>
   </joint>
   <joint name="rear_left_steering_joint" type="continuous">
@@ -183,4 +191,5 @@
     <origin xyz="-0.58 0.275 0" rpy="0 0 0"/>
     <axis xyz="0 0 1"/>
+    <dynamics damping="5.0" friction="0.1"/>
   </joint>
   <joint name="rear_right_steering_joint" type="continuous">
@@ -189,4 +198,5 @@
     <origin xyz="-0.58 -0.275 0" rpy="0 0 0"/>
     <axis xyz="0 0 1"/>
+    <dynamics damping="5.0" friction="0.1"/>
   </joint>
   <!-- Wheel Links -->
